Commit message: cambios en las dependencias del las mallas

File: irb140_layout/urdf/irb140_gripper.urdf (robot description, URDF)
Before this commit: robot irb140_robot, 16 links, 15 joints
Links:
- link base_link: geometry collision mesh filename=package://irb140_layout/meshes/irb140/collision_low_poly/ba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 scale=0.01 0.01 0.01; visual mesh filename=package://irb140_layout/meshes/irb140/visual/base_link.stl scale=0.01 0.01 0.01
